File: DivMMC.kicad_sch (KiCad schematic)
At the start: 30 parts, among them J12 Header 5x2, J13 693063020911, J14 uSD Card Socket ST-TF-003A, J15 Header 3x2, J16 Header 2x1, Q2 Transistor BC548, U16 EPM7128SLC84-10, U17 EEPROM 8Kx8 AT28C64B-15PU, U18 AS6C1008-55PCN, U19 3V3 1Amp

Commit message: Add files via upload
Latest additions to include full track routing and vias to allow a full ibom to be created. Part 3. While Kicad created the gerbers without error I am not convinced about getting any pcbs manufactured without someone else verifying the created schematics against the originals from DonSuperFo and then verifying that schematic against the pcb layout. I only did this as an exercise to create a full ibom to assist in component assembly.
Parts:
- J13: value 693063020911 -> Wurth 693063020911; footprint 693063020911 -> Mod:SD Card Connector Wurth 693063020911
