File: ZX Max 128 Issue 5 PCB.kicad_pcb (KiCad board)
At the start: 2 copper layers, 213 x 130 mm, 262 parts, among them J1 8 Pin FFC Connector, J10 Header 2x1, J11 Header 2x1, J12 Header 5x2, J13 SD Card Socket, J14 uSD Card Socket ST-TF-003A, J15 Header 3x2, J16 Header 2x1, J17 Header 2x1, J2 5 Pin FFC Connector, J3 ZX_48K_EDGE, J4 PJ-002A, J5 AV Jack, J6 Connector Audio 3525N, J7 A-DS_09_A_KG-T4S, J8 Connector 9 Pin Mini DIN, J9 Header 5x2, M1 MountingHole, M2 MountingHole, M3 MountingHole, M4 MountingHole, M5 MountingHole, M6 MountingHole, Q1 Transistor BC548, Q2 Transistor BC548, U1 Z80, U10 CD74HC30E, U11 74HC74, U12 CD74HC366E, U13 AD724JRZ, U14 R-78E5.0-1.0, U15 ESP8266-12E, U16 EPM7128SLC84-10, U17 EEPROM 8Kx8 AT28C64B-15PU, U18 AS6C1008-55PCN, U19 3V3 1Amp, U2 EEPROM/EPROM 32Kx8, U20 CD74HC30E, U21 74HC32, U22 Sound Generator SAA1099, U23 MCP602-E_SN, U24 SAM2695, U25 3V3 1Amp, U3 AS6C1008-55PCN, U4 AS6C1008-55PCN, U5 EPM7128SLC, U6 74HC04, U7 SN74HC174N, U8 AY-3-8910, U9 AY-3-8910, Y1 28.375Mhz, Y2 4.433Mhz, Y3 ECS-2100A-080, Y4 12Mhz

Commit message: Add files via upload
Latest additions to include full track routing and vias to allow a full ibom to be created. Part 3. While Kicad created the gerbers without error I am not convinced about getting any pcbs manufactured without someone else verifying the created schematics against the originals from DonSuperFo and then verifying that schematic against the pcb layout. I only did this as an exercise to create a full ibom to assist in component assembly.
Parts:
- J13: value SD Card Socket -> Wurth 693063020911
- moved J13 0.14 mm to (220.0, 125.4)
Routing:
- net GND: track 0.00 -> 1573.9 mm, vias 0 -> 11
- net VCC: track 0.00 -> 1018.1 mm, vias 0 -> 5
- net D4: track 0.00 -> 462.7 mm, vias 0 -> 10
- net RST: track 0.00 -> 455.8 mm, vias 0 -> 12
- net D3: track 0.00 -> 446.9 mm, vias 0 -> 12
- net D1: track 0.00 -> 438.8 mm, vias 0 -> 8
- net D0: track 0.00 -> 428.1 mm, vias 0 -> 8
- net IORQ: track 0.00 -> 412.6 mm, vias 0 -> 9
- net WR: track 0.00 -> 411.7 mm, vias 0 -> 5
- net A1: track 0.00 -> 386.1 mm, vias 0 -> 9
- net D5: track 0.00 -> 374.4 mm, vias 0 -> 7
- net D7: track 0.00 -> 361.6 mm, vias 0 -> 7
- net D2: track 0.00 -> 360.3 mm, vias 0 -> 8
- net A4: track 0.00 -> 351.0 mm, vias 0 -> 7
- net A14: track 0.00 -> 343.5 mm, vias 0 -> 10
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- added copper zone on B.Cu, net GND
- added copper zone on F.Cu, net VCC
